File: Documentation/pcbDesign/adafruitBuck/Adafruit MPM3610.kicad_sch (KiCad schematic)
At the start: 9 parts, among them IC1 MPM3610

Commit message: Verified circuit. Time to finalize Schematic with symbols that have compatible footprints. Need to add remaining 3D models, testing pins for PCB, and verify relay octocoupler footprint + symbol
Parts:
- removed C1, C2: 22uF, buckConverter:0805-NO, symbol buckConverter-eagle-import:CAP_CERAMIC0805-NOOUTLINE
- removed FID1: FIDUCIAL_1MM, buckConverter:FIDUCIAL_1MM, symbol buckConverter-eagle-import:FIDUCIAL_1MM
- removed IC1: MPM3610, buckConverter:MPM3610, symbol buckConverter-eagle-import:MPM3610
- removed JP1: HEADER-1X4ROUND, buckConverter:1X04_ROUND, symbol buckConverter-eagle-import:HEADER-1X4ROUND
- removed R1, R2: 75K, buckConverter:0603-NO, symbol buckConverter-eagle-import:RESISTOR_0603_NOOUT
- removed R3: 24K, buckConverter:0603-NO, symbol buckConverter-eagle-import:RESISTOR_0603_NOOUT
- removed U$9: MOUNTINGHOLE2.5, buckConverter:MOUNTINGHOLE_2.5_PLATED, symbol buckConverter-eagle-import:MOUNTINGHOLE2.5
- added C1, C2: 22uF, Adafruit MPM3610:0805-NO, symbol Adafruit MPM3610-eagle-import:CAP_CERAMIC0805-NOOUTLINE
- added FID1: FIDUCIAL_1MM, Adafruit MPM3610:FIDUCIAL_1MM, symbol Adafruit MPM3610-eagle-import:FIDUCIAL_1MM
- added IC1: MPM3610, Adafruit MPM3610:MPM3610, symbol Adafruit MPM3610-eagle-import:MPM3610
- added JP1: HEADER-1X4ROUND, Adafruit MPM3610:1X04_ROUND, symbol Adafruit MPM3610-eagle-import:HEADER-1X4ROUND
- added R1, R2: 75K, Adafruit MPM3610:0603-NO, symbol Adafruit MPM3610-eagle-import:RESISTOR_0603_NOOUT
- added R3: 24K, Adafruit MPM3610:0603-NO, symbol Adafruit MPM3610-eagle-import:RESISTOR_0603_NOOUT
- added U$9: MOUNTINGHOLE2.5, Adafruit MPM3610:MOUNTINGHOLE_2.5_PLATED, symbol Adafruit MPM3610-eagle-import:MOUNTINGHOLE2.5
Connections:
- net 3.3V: now also C1.1, IC1.7 (OUT), IC1.8 (OUT), IC1.9 (OUT), JP1.3, R2.1
- net EN: now also IC1.17 (EN), JP1.1, R1.2
- net FB: now also IC1.1 (FB), R2.2, R3.1
- net GND: now also C1.2, C2.2, IC1.12 (PGND), IC1.13 (PGND), IC1.14 (PGND), IC1.3 (AGND), JP1.4, R3.2
- net SW: now also IC1.4 (SW), IC1.5 (SW), IC1.6 (SW)
- net VCC: now also IC1.2 (VCC)
- net VIN: now also C2.1, IC1.16 (IN), JP1.2, R1.1
