File: Documentation/pcbDesign/plantPartner_PCB1.0/plantPartner_PCB1.0.kicad_pcb (KiCad board)
At the start: 2 copper layers, 271 x 152 mm, 76 parts, among them IC1 MPM3610, J1 Conn_01x04, J10 Screw_Terminal_01x03, J11 Conn_01x04, J12 Conn_01x03, J13 Conn_01x03, J14 Conn_01x03, J15 Conn_01x03, J16 Conn_01x04, J17 Conn_01x03, J18 Screw_Terminal_01x02, J19 Barrel_Jack, J2 Conn_01x04, J20 Conn_02x04_Top_Bottom, J21 Conn_01x04, J22 Conn_01x04, J23 Conn_01x02, J24 Conn_01x04, J25 Conn_01x04, J26 Conn_01x01, J27 Conn_01x03, J3 Conn_01x04, J4 Screw_Terminal, J5 Conn_01x02, J6 Screw_Terminal_01x03, J7 Conn_01x03, J8 Conn_02x04_Top_Bottom, J9 Conn_01x03, K1 SRD-05VDC-SL-C, K2 SRD-05VDC-SL-C, Q1 PNP, Q2 PNP, U1 EL357N-G, U2 MAX485, U3 ESP32-DEVKIT-V1, U4 EL357N-G

Commit message: Routed the 5V Relays and fixed a schematic issue I made with them. Next is the Buck Converter, RS485 Transceiver, Power Supplies, and ESP32 Signals
Parts:
- moved D7 219.0 mm to (243.6, 101.9), turned to 180 degrees
- moved D4 194.4 mm to (56.5, 109.0), turned to 180 degrees
- moved J27 105.6 mm to (136.0, 41.2)
- moved J26 48.7 mm to (277.4, 159.6)
- moved J14 42.6 mm to (69.3, 105.2), turned to 180 degrees
- moved U4 42.6 mm to (240.8, 112.7)
- moved J7 39.8 mm to (63.2, 91.5), turned to 90 degrees
- moved R18 34.4 mm to (238.0, 109.9), turned to 180 degrees
- moved J8 32.2 mm to (66.8, 154.6)
- moved R19 32.0 mm to (244.3, 110.0), turned to 180 degrees
- moved R17 31.8 mm to (238.3, 105.5), turned to 180 degrees
- moved J13 31.0 mm to (261.3, 116.8), turned to -90 degrees
- moved J9 30.7 mm to (243.2, 117.1), turned to -90 degrees
- moved R20 29.5 mm to (244.3, 109.2)
- moved Q2 27.9 mm to (243.3, 105.7), turned to 180 degrees
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Connections:
- net /<NO NET> renamed /ADC2_3/Touch3
- J10 pad 1: GND -> /COM
- J10 pad 2: /NO -> /NC
- J10 pad 3: /COM -> GND
- J13 pad 1: /NO -> +12V
- J13 pad 3: +12V -> /NC
- J15 pad 1: /NO -> +12V
- J15 pad 3: +12V -> /NC
- J6 pad 1: GND -> /COM
- J6 pad 2: /NO -> /NC
- J6 pad 3: /COM -> GND
- J7 pad 2: Net-(J7-Pin_2) -> /H
- J9 pad 2: Net-(J9-Pin_2) -> /H
- K1 pad NC: +12V -> /NC
- K1 pad NO: /NO -> +12V
- K2 pad NC: +12V -> /NC
- K2 pad NO: /NO -> +12V
- R13 pad 1: Net-(J7-Pin_2) -> /H
- R18 pad 1: Net-(J9-Pin_2) -> /H
Routing:
- net /COM: track 0.00 -> 70.9 mm
- net GND: track 32.9 -> 95.1 mm
- net /NC: track 0.00 -> 53.4 mm
- net +5V: track 0.91 -> 28.1 mm
- net +12V: track 26.9 -> 44.1 mm
- net Net-(D7-K): track 0.00 -> 11.9 mm
- net Net-(D4-K): track 0.00 -> 11.6 mm
- net /H: track 0.00 -> 8.19 mm
- net Net-(R14-Pad2): track 0.00 -> 5.77 mm
- net Net-(Q2-B): track 0.00 -> 3.60 mm
- net Net-(R19-Pad2): track 0.00 -> 2.28 mm
- net Net-(Q1-B): track 0.00 -> 2.03 mm
- net Net-(R18-Pad2): track 0.00 -> 1.64 mm
- net Net-(R13-Pad2): track 0.00 -> 1.54 mm
- net Net-(D3-A): track 0.00 -> 0.88 mm
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Other:
- board text added: "+12V"
- board text added: "+5V"
- board text added: "+5V H GND"
- board text added: "5V Relay - Fertilizer Pump"
- board text added: "5V Relay - Water Pump"
- board text added: "COM"
- board text added: "GND"
- board text added: "GND H +5V"
- board text added: "NC"
- board text added: "NC COM +12V"
